File: Battery_Monitoring_System_Drawing/BMS/Analog_Measurements.sch (KiCad schematic (older format))
At the start: 14 parts, among them J4 Conn_01x04, J5 ACS INPUT, U5 ACS712xLCTR-30A

Commit message: Layout çizimi tamanlandı.
Layout çizimi ilk şablonu tamamlandı.
Parts:
- J5: footprint Connector_Phoenix_MSTB:PhoenixContact_MSTBA_2,5_2-G_1x02_P5.00mm_Horizontal -> TerminalBlock_Phoenix:TerminalBlock_Phoenix_MKDS-1,5-2_1x02_P5.00mm_Horizontal
- renumbered C21 to C22, C22 to C23, R11 to R10, R12 to R11, R14 to R12, R15 to R14, R16 to R15, R17 to R16
Other:
- moved on the sheet: R10, R11, R12, R14
Changed lines of the file:
@@
 P 1950 3750
 AR Path="/609D1626" Ref="#PWR?"  Part="1"
-AR Path="/609AC84F/609D1626" Ref="#PWR038"  Part="1"
-F 0 "#PWR038" H 1950 3500 50  0001 C CNN
+AR Path="/609AC84F/609D1626" Ref="#PWR037"  Part="1"
+F 0 "#PWR037" H 1950 3500 50  0001 C CNN
 F 1 "GND" H 1955 3577 50  0000 C CNN
 F 2 "" H 1950 3750 50  0001 C CNN
@@
 Wire Wire Line
 	1950 3350 1950 3450
-Text Label 1650 3350 0    50   ~ 0
-NTC
 $Comp
 L Sensor_Current:ACS712xLCTR-30A U?
@@
 P 6250 2750
 AR Path="/609D1637" Ref="C?"  Part="1"
-AR Path="/609AC84F/609D1637" Ref="C22"  Part="1"
-F 0 "C22" H 6365 2796 50  0000 L CNN
+AR Path="/609AC84F/609D1637" Ref="C23"  Part="1"
+F 0 "C23" H 6365 2796 50  0000 L CNN
 F 1 "1nF" H 6365 2705 50  0000 L CNN
 F 2 "Capacitor_SMD:C_0805_2012Metric" H 6288 2600 50  0001 C CNN
@@
 P 6150 1800
 AR Path="/609D163D" Ref="C?"  Part="1"
-AR Path="/609AC84F/609D163D" Ref="C21"  Part="1"
-F 0 "C21" V 5898 1800 50  0000 C CNN
+AR Path="/609AC84F/609D163D" Ref="C22"  Part="1"
+F 0 "C22" V 5898 1800 50  0000 C CNN
 F 1 "100nF" V 5989 1800 50  0000 C CNN
 F 2 "Capacitor_SMD:C_0805_2012Metric" H 6188 1650 50  0001 C CNN
@@
 P 6400 1800
 AR Path="/609D164B" Ref="#PWR?"  Part="1"
-AR Path="/609AC84F/609D164B" Ref="#PWR045"  Part="1"
-F 0 "#PWR045" H 6400 1550 50  0001 C CNN
+AR Path="/609AC84F/609D164B" Ref="#PWR043"  Part="1"
+F 0 "#PWR043" H 6400 1550 50  0001 C CNN
 F 1 "GND" H 6405 1627 50  0000 C CNN
 F 2 "" H 6400 1800 50  0001 C CNN
@@
 P 5750 3050
 AR Path="/609D1651" Ref="#PWR?"  Part="1"
-AR Path="/609AC84F/609D1651" Ref="#PWR043"  Part="1"
-F 0 "#PWR043" H 5750 2800 50  0001 C CNN
+AR Path="/609AC84F/609D1651" Ref="#PWR041"  Part="1"
+F 0 "#PWR041" H 5750 2800 50  0001 C CNN
 F 1 "GND" H 5755 2877 50  0000 C CNN
 F 2 "" H 5750 3050 50  0001 C CNN
@@
 P 5350 1450
 AR Path="/609D1660" Ref="#PWR?"  Part="1"
-AR Path="/609AC84F/609D1660" Ref="#PWR042"  Part="1"
-F 0 "#PWR042" H 5350 1300 50  0001 C CNN
+AR Path="/609AC84F/609D1660" Ref="#PWR040"  Part="1"
+F 0 "#PWR040" H 5350 1300 50  0001 C CNN
 F 1 "+5V" H 5365 1623 50  0000 C CNN
 F 2 "" H 5350 1450 50  0001 C CNN
@@
 F 0 "J5" H 4668 2125 50  0000 C CNN
 F 1 "ACS INPUT" H 4668 2216 50  0000 C CNN
-F 2 "Connector_Phoenix_MSTB:PhoenixContact_MSTBA_2,5_2-G_1x02_P5.00mm_Horizontal" H 4750 2450 50  0001 C CNN
+F 2 "TerminalBlock_Phoenix:TerminalBlock_Phoenix_MKDS-1,5-2_1x02_P5.00mm_Horizontal" H 4750 2450 50  0001 C CNN
 F 3 "~" H 4750 2450 50  0001 C CNN
 	1    4750 2450
@@
 Wire Wire Line
 	5150 2600 5350 2600
-Text Label 5250 1800 0    50   ~ 0
-ACS_SUPPLY
 Connection ~ 5750 1800
 Wire Wire Line
@@
 Wire Wire Line
 	5750 1800 5250 1800
-Text Label 6300 2400 0    50   ~ 0
-ACS_OUT
 Wire Wire Line
 	6150 2400 6300 2400
@@
 P 1950 2950
 AR Path="/609D167F" Ref="#PWR?"  Part="1"
-AR Path="/609AC84F/609D167F" Ref="#PWR037"  Part="1"
-F 0 "#PWR037" H 1950 2800 50  0001 C CNN
+AR Path="/609AC84F/609D167F" Ref="#PWR036"  Part="1"
+F 0 "#PWR036" H 1950 2800 50  0001 C CNN
 F 1 "+5V" H 1965 3123 50  0000 C CNN
 F 2 "" H 1950 2950 50  0001 C CNN
@@
 $EndComp
 $Comp
-L power:+3.3VA #PWR044
+L power:+3.3VA #PWR042
 U 1 1 60A3BC96
 P 6150 1450
-F 0 "#PWR044" H 6150 1300 50  0001 C CNN
+F 0 "#PWR042" H 6150 1300 50  0001 C CNN
 F 1 "+3.3VA" H 6165 1623 50  0000 C CNN
 F 2 "" H 6150 1450 50  0001 C CNN
@@
 L Device:R_Small R?
 U 1 1 60B09032
-P 2000 1700
+P 1950 1700
 AR Path="/60B09032" Ref="R?"  Part="1"
-AR Path="/609AC84F/60B09032" Ref="R14"  Part="1"
-F 0 "R14" H 2059 1746 50  0000 L CNN
-F 1 "12K" H 2059 1655 50  0000 L CNN
-F 2 "Resistor_SMD:R_0805_2012Metric" H 2000 1700 50  0001 C CNN
-F 3 "~" H 2000 1700 50  0001 C CNN
-	1    2000 1700
+AR Path="/609AC84F/60B09032" Ref="R12"  Part="1"
+F 0 "R12" H 2009 1746 50  0000 L CNN
+F 1 "12K" H 2009 1655 50  0000 L CNN
+F 2 "Resistor_SMD:R_0805_2012Metric" H 1950 1700 50  0001 C CNN
+F 3 "~" H 1950 1700 50  0001 C CNN
+	1    1950 1700
 	1    0    0    -1
 $EndComp
@@
 L Device:R_Small R?
 U 1 1 60B09038
-P 1350 1700
+P 1250 1700
 AR Path="/60B09038" Ref="R?"  Part="1"
-AR Path="/609AC84F/60B09038" Ref="R11"  Part="1"
-F 0 "R11" H 1409 1746 50  0000 L CNN
-F 1 "12K" H 1409 1655 50  0000 L CNN
-F 2 "Resistor_SMD:R_0805_2012Metric" H 1350 1700 50  0001 C CNN
-F 3 "~" H 1350 1700 50  0001 C CNN
-	1    1350 1700
+AR Path="/609AC84F/60B09038" Ref="R10"  Part="1"
+F 0 "R10" H 1309 1746 50  0000 L CNN
+F 1 "12K" H 1309 1655 50  0000 L CNN
+F 2 "Resistor_SMD:R_0805_2012Metric" H 1250 1700 50  0001 C CNN
+F 3 "~" H 1250 1700 50  0001 C CNN
+	1    1250 1700
 	1    0    0    -1
 $EndComp
@@
 L Device:R_Small R?
 U 1 1 60B0903E
-P 1500 1250
+P 1400 1250
 AR Path="/60B0903E" Ref="R?"  Part="1"
-AR Path="/609AC84F/60B0903E" Ref="R12"  Part="1"
-F 0 "R12" V 1450 1400 50  0000 C CNN
-F 1 "3.3K" V 1550 1400 50  0000 C CNN
-F 2 "Resistor_SMD:R_0805_2012Metric" H 1500 1250 50  0001 C CNN
-F 3 "~" H 1500 1250 50  0001 C CNN
-	1    1500 1250
+AR Path="/609AC84F/60B0903E" Ref="R11"  Part="1"
+F 0 "R11" V 1350 1400 50  0000 C CNN
+F 1 "3.3K" V 1450 1400 50  0000 C CNN
+F 2 "Resistor_SMD:R_0805_2012Metric" H 1400 1250 50  0001 C CNN
+F 3 "~" H 1400 1250 50  0001 C CNN
+	1    1400 1250
 	0    1    1    0
 $EndComp
@@
 L Device:R_Small R?
 U 1 1 60B09044
-P 2150 1350
+P 2100 1350
 AR Path="/60B09044" Ref="R?"  Part="1"
-AR Path="/609AC84F/60B09044" Ref="R15"  Part="1"
-F 0 "R15" V 2100 1500 50  0000 C CNN
-F 1 "22K" V 2200 1500 50  0000 C CNN
-F 2 "Resistor_SMD:R_0805_2012Metric" H 2150 1350 50  0001 C CNN
-F 3 "~" H 2150 1350 50  0001 C CNN
-	1    2150 1350
+AR Path="/609AC84F/60B09044" Ref="R14"  Part="1"
+F 0 "R14" V 2050 1500 50  0000 C CNN
+F 1 "22K" V 2150 1500 50  0000 C CNN
+F 2 "Resistor_SMD:R_0805_2012Metric" H 2100 1350 50  0001 C CNN
+F 3 "~" H 2100 1350 50  0001 C CNN
+	1    2100 1350
 	0    1    1    0
 $EndComp
@@
 P 2650 1700
 AR Path="/60B0904A" Ref="R?"  Part="1"
-AR Path="/609AC84F/60B0904A" Ref="R16"  Part="1"
-F 0 "R16" H 2709 1746 50  0000 L CNN
+AR Path="/609AC84F/60B0904A" Ref="R15"  Part="1"
+F 0 "R15" H 2709 1746 50  0000 L CNN
 F 1 "22K" H 2709 1655 50  0000 L CNN
 F 2 "Resistor_SMD:R_0805_2012Metric" H 2650 1700 50  0001 C CNN
@@
 P 2800 1450
 AR Path="/60B09050" Ref="R?"  Part="1"
-AR Path="/609AC84F/60B09050" Ref="R17"  Part="1"
-F 0 "R17" V 2750 1600 50  0000 C CNN
+AR Path="/609AC84F/60B09050" Ref="R16"  Part="1"
+F 0 "R16" V 2750 1600 50  0000 C CNN
 F 1 "68K" V 2850 1600 50  0000 C CNN
 F 2 "Resistor_SMD:R_0805_2012Metric" H 2800 1450 50  0001 C CNN
@@
 	3000 1450 2900 1450
 Wire Wire Line
-	1400 1250 1350 1250
-Wire Wire Line
-	1350 1250 1350 1600
-Wire Wire Line
-	2050 1350 2000 1350
-Wire Wire Line
-	2000 1350 2000 1600
+	1300 1250 1250 1250
+Wire Wire Line
+	1250 1250 1250 1600
+Wire Wire Line
+	2000 1350 1950 1350
+Wire Wire Line
+	1950 1350 1950 1600
 Wire Wire Line
 	2700 1450 2650 1450
@@
 P 3000 1150
 AR Path="/60B0905D" Ref="#PWR?"  Part="1"
-AR Path="/609AC84F/60B0905D" Ref="#PWR041"  Part="1"
-F 0 "#PWR041" H 3000 900 50  0001 C CNN
+AR Path="/609AC84F/60B0905D" Ref="#PWR039"  Part="1"
+F 0 "#PWR039" H 3000 900 50  0001 C CNN
 F 1 "GND" V 3005 1022 50  0000 R CNN
 F 2 "" H 3000 1150 50  0001 C CNN
@@
 P 2650 1800
 AR Path="/60B09063" Ref="#PWR?"  Part="1"
-AR Path="/609AC84F/60B09063" Ref="#PWR040"  Part="1"
-F 0 "#PWR040" H 2650 1550 50  0001 C CNN
+AR Path="/609AC84F/60B09063" Ref="#PWR038"  Part="1"
+F 0 "#PWR038" H 2650 1550 50  0001 C CNN
 F 1 "GND" H 2655 1627 50  0000 C CNN
 F 2 "" H 2650 1800 50  0001 C CNN
@@
 L power:GND #PWR?
 U 1 1 60B09069
-P 2000 1800
+P 1950 1800
 AR Path="/60B09069" Ref="#PWR?"  Part="1"
-AR Path="/609AC84F/60B09069" Ref="#PWR039"  Part="1"
-F 0 "#PWR039" H 2000 1550 50  0001 C CNN
-F 1 "GND" H 2005 1627 50  0000 C CNN
-F 2 "" H 2000 1800 50  0001 C CNN
-F 3 "" H 2000 1800 50  0001 C CNN
-	1    2000 1800
+AR Path="/609AC84F/60B09069" Ref="#PWR035"  Part="1"
+F 0 "#PWR035" H 1950 1550 50  0001 C CNN
+F 1 "GND" H 1955 1627 50  0000 C CNN
+F 2 "" H 1950 1800 50  0001 C CNN
+F 3 "" H 1950 1800 50  0001 C CNN
+	1    1950 1800
 	1    0    0    -1
 $EndComp
@@
 L power:GND #PWR?
 U 1 1 60B0906F
-P 1350 1800
+P 1250 1800
 AR Path="/60B0906F" Ref="#PWR?"  Part="1"
-AR Path="/609AC84F/60B0906F" Ref="#PWR036"  Part="1"
-F 0 "#PWR036" H 1350 1550 50  0001 C CNN
-F 1 "GND" H 1355 1627 50  0000 C CNN
-F 2 "" H 1350 1800 50  0001 C CNN
-F 3 "" H 1350 1800 50  0001 C CNN
-	1    1350 1800
-	1    0    0    -1
-$EndComp
-Text Label 2650 1450 2    50   ~ 0
+AR Path="/609AC84F/60B0906F" Ref="#PWR034"  Part="1"
+F 0 "#PWR034" H 1250 1550 50  0001 C CNN
+F 1 "GND" H 1255 1627 50  0000 C CNN
+F 2 "" H 1250 1800 50  0001 C CNN
+F 3 "" H 1250 1800 50  0001 C CNN
+	1    1250 1800
+	1    0    0    -1
+$EndComp
+Text GLabel 2650 1450 0    50   Input ~ 0
 CELL_1
 Wire Wire Line
-	2250 1350 3000 1350
-Text Label 2000 1350 2    50   ~ 0
+	2200 1350 3000 1350
+Text GLabel 1950 1350 0    50   Input ~ 0
 CELL_2
 Wire Wire Line
-	1600 1250 3000 1250
-Text Label 1350 1250 2    50   ~ 0
+	1500 1250 3000 1250
+Text GLabel 1250 1250 0    50   Input ~ 0
 CELL_3
+Text GLabel 1650 3350 0    50   Input ~ 0
+NTC
+Text GLabel 5250 1800 0    50   Input ~ 0
+ACS_SUPPLY
+Text GLabel 6300 2400 2    50   Input ~ 0
+ACS_OUT
 $EndSCHEMATC

Commit message: Micro Sd kılıf eklendi.
Sd kart holder kılıfı micro sd kart soket kılıfı ile değiştirildi.
Parts:
- renumbered C22 to C20, C23 to C21
Changed lines of the file:
@@
 P 1950 3750
 AR Path="/609D1626" Ref="#PWR?"  Part="1"
-AR Path="/609AC84F/609D1626" Ref="#PWR037"  Part="1"
-F 0 "#PWR037" H 1950 3500 50  0001 C CNN
+AR Path="/609AC84F/609D1626" Ref="#PWR036"  Part="1"
+F 0 "#PWR036" H 1950 3500 50  0001 C CNN
 F 1 "GND" H 1955 3577 50  0000 C CNN
 F 2 "" H 1950 3750 50  0001 C CNN
@@
 P 6250 2750
 AR Path="/609D1637" Ref="C?"  Part="1"
-AR Path="/609AC84F/609D1637" Ref="C23"  Part="1"
-F 0 "C23" H 6365 2796 50  0000 L CNN
+AR Path="/609AC84F/609D1637" Ref="C21"  Part="1"
+F 0 "C21" H 6365 2796 50  0000 L CNN
 F 1 "1nF" H 6365 2705 50  0000 L CNN
 F 2 "Capacitor_SMD:C_0805_2012Metric" H 6288 2600 50  0001 C CNN
@@
 P 6150 1800
 AR Path="/609D163D" Ref="C?"  Part="1"
-AR Path="/609AC84F/609D163D" Ref="C22"  Part="1"
-F 0 "C22" V 5898 1800 50  0000 C CNN
+AR Path="/609AC84F/609D163D" Ref="C20"  Part="1"
+F 0 "C20" V 5898 1800 50  0000 C CNN
 F 1 "100nF" V 5989 1800 50  0000 C CNN
 F 2 "Capacitor_SMD:C_0805_2012Metric" H 6188 1650 50  0001 C CNN
@@
 P 6400 1800
 AR Path="/609D164B" Ref="#PWR?"  Part="1"
-AR Path="/609AC84F/609D164B" Ref="#PWR043"  Part="1"
-F 0 "#PWR043" H 6400 1550 50  0001 C CNN
+AR Path="/609AC84F/609D164B" Ref="#PWR042"  Part="1"
+F 0 "#PWR042" H 6400 1550 50  0001 C CNN
 F 1 "GND" H 6405 1627 50  0000 C CNN
 F 2 "" H 6400 1800 50  0001 C CNN
@@
 P 5750 3050
 AR Path="/609D1651" Ref="#PWR?"  Part="1"
-AR Path="/609AC84F/609D1651" Ref="#PWR041"  Part="1"
-F 0 "#PWR041" H 5750 2800 50  0001 C CNN
+AR Path="/609AC84F/609D1651" Ref="#PWR040"  Part="1"
+F 0 "#PWR040" H 5750 2800 50  0001 C CNN
 F 1 "GND" H 5755 2877 50  0000 C CNN
 F 2 "" H 5750 3050 50  0001 C CNN
@@
 P 5350 1450
 AR Path="/609D1660" Ref="#PWR?"  Part="1"
-AR Path="/609AC84F/609D1660" Ref="#PWR040"  Part="1"
-F 0 "#PWR040" H 5350 1300 50  0001 C CNN
+AR Path="/609AC84F/609D1660" Ref="#PWR039"  Part="1"
+F 0 "#PWR039" H 5350 1300 50  0001 C CNN
 F 1 "+5V" H 5365 1623 50  0000 C CNN
 F 2 "" H 5350 1450 50  0001 C CNN
@@
 P 1950 2950
 AR Path="/609D167F" Ref="#PWR?"  Part="1"
-AR Path="/609AC84F/609D167F" Ref="#PWR036"  Part="1"
-F 0 "#PWR036" H 1950 2800 50  0001 C CNN
+AR Path="/609AC84F/609D167F" Ref="#PWR035"  Part="1"
+F 0 "#PWR035" H 1950 2800 50  0001 C CNN
 F 1 "+5V" H 1965 3123 50  0000 C CNN
 F 2 "" H 1950 2950 50  0001 C CNN
@@
 $EndComp
 $Comp
-L power:+3.3VA #PWR042
+L power:+3.3VA #PWR041
 U 1 1 60A3BC96
 P 6150 1450
-F 0 "#PWR042" H 6150 1300 50  0001 C CNN
+F 0 "#PWR041" H 6150 1300 50  0001 C CNN
 F 1 "+3.3VA" H 6165 1623 50  0000 C CNN
 F 2 "" H 6150 1450 50  0001 C CNN
@@
 P 3000 1150
 AR Path="/60B0905D" Ref="#PWR?"  Part="1"
-AR Path="/609AC84F/60B0905D" Ref="#PWR039"  Part="1"
-F 0 "#PWR039" H 3000 900 50  0001 C CNN
+AR Path="/609AC84F/60B0905D" Ref="#PWR038"  Part="1"
+F 0 "#PWR038" H 3000 900 50  0001 C CNN
 F 1 "GND" V 3005 1022 50  0000 R CNN
 F 2 "" H 3000 1150 50  0001 C CNN
@@
 P 2650 1800
 AR Path="/60B09063" Ref="#PWR?"  Part="1"
-AR Path="/609AC84F/60B09063" Ref="#PWR038"  Part="1"
-F 0 "#PWR038" H 2650 1550 50  0001 C CNN
+AR Path="/609AC84F/60B09063" Ref="#PWR037"  Part="1"
+F 0 "#PWR037" H 2650 1550 50  0001 C CNN
 F 1 "GND" H 2655 1627 50  0000 C CNN
 F 2 "" H 2650 1800 50  0001 C CNN
@@
 P 1950 1800
 AR Path="/60B09069" Ref="#PWR?"  Part="1"
-AR Path="/609AC84F/60B09069" Ref="#PWR035"  Part="1"
-F 0 "#PWR035" H 1950 1550 50  0001 C CNN
+AR Path="/609AC84F/60B09069" Ref="#PWR034"  Part="1"
+F 0 "#PWR034" H 1950 1550 50  0001 C CNN
 F 1 "GND" H 1955 1627 50  0000 C CNN
 F 2 "" H 1950 1800 50  0001 C CNN
@@
 P 1250 1800
 AR Path="/60B0906F" Ref="#PWR?"  Part="1"
-AR Path="/609AC84F/60B0906F" Ref="#PWR034"  Part="1"
-F 0 "#PWR034" H 1250 1550 50  0001 C CNN
+AR Path="/609AC84F/60B0906F" Ref="#PWR033"  Part="1"
+F 0 "#PWR033" H 1250 1550 50  0001 C CNN
 F 1 "GND" H 1255 1627 50  0000 C CNN
 F 2 "" H 1250 1800 50  0001 C CNN
