File: Battery_Monitoring_System_Drawing/BMS/BMS.sch (KiCad schematic (older format))
At the start: 35 parts, among them U1 STM32F101C8Tx

Commit message: Şematik çizimi tamamlandı.
Şematik çizimi ve footprint  atamaları tamamlandı.
Parts:
- removed C?: 1nF, symbol Device:C
- removed C?: 100nF, symbol Device:C
- removed J?: SW Pins, symbol Connector:Conn_01x03_Male
- removed J?: ACS INPUT, symbol Connector_Generic:Conn_01x02
- removed JP?: ACS SUPPLY, symbol Jumper:Jumper_3_Bridged12
- removed R?: 10K, symbol Device:R
- removed TH?: NTC_10K, symbol Device:Thermistor_NTC
- removed U?: ACS712xLCTR-30A, Package_SO:SOIC-8_3.9x4.9mm_P1.27mm, symbol Sensor_Current:ACS712xLCTR-30A
- added C14, C6: 10uF, Capacitor_SMD:C_0805_2012Metric, symbol Device:CP_Small
- added C16, C9: 100nF, Capacitor_SMD:C_0805_2012Metric, symbol Device:C_Small
- added C19, C20: 100nF, Capacitor_SMD:C_0805_2012Metric, symbol Device:C
- added C23: 10uF, Capacitor_SMD:C_0805_2012Metric, symbol Device:C
- added D3: LED, LED_SMD:LED_0805_2012Metric, symbol Device:LED
- added D4: SD CARD LED, LED_SMD:LED_0805_2012Metric, symbol Device:LED
- added J1: SWD Pins, Connector_JST:JST_XH_B3B-XH-A_1x03_P2.50mm_Vertical, symbol Connector_Generic:Conn_01x03
- added J3: Micro_SD_Card_Det_Hirose_DM3AT, Connector_Card:SD_Kyocera_145638009511859+, symbol Connector:Micro_SD_Card_Det_Hirose_DM3AT
- added JP2: ESP BOOT JUMPER, Connector_PinHeader_2.54mm:PinHeader_1x03_P2.54mm_Vertical, symbol Jumper:Jumper_3_Bridged12
- added R10, R7, R8, R9: 10K, Resistor_SMD:R_0805_2012Metric, symbol Device:R_Small
- added R4, R6: 470, Resistor_SMD:R_0805_2012Metric, symbol Device:R_Small
- added SW2: ESP RESET BUTTON, Button_Switch_THT:SW_PUSH_6mm_H5mm, symbol Switch:SW_Push_Dual
- added U2: AMS1117-3.3, Package_TO_SOT_SMD:SOT-223-3_TabPin2, symbol Regulator_Linear:AMS1117-3.3
- added U4: ESP-12E, RF_Module:ESP-12E, symbol RF_Module:ESP-12E
- C1, C11, C12, C13, C15, C18, C2, C3, C4, C5, C7, C8: renamed from C?; footprint (none) -> Capacitor_SMD:C_0805_2012Metric
- C10, C17: renamed from C?; value 0.1uF -> 100nF; footprint (none) -> Capacitor_SMD:C_0805_2012Metric
- D1, D2: renamed from D?; footprint (none) -> LED_SMD:LED_0805_2012Metric
- J2: renamed from J?; footprint (none) -> Connector_JST:JST_XH_B2B-XH-A_1x02_P2.50mm_Vertical
- JP1: renamed from JP?; footprint (none) -> Connector_PinHeader_2.54mm:PinHeader_1x03_P2.54mm_Vertical
- R1, R2, R3, R5: renamed from R?; footprint (none) -> Resistor_SMD:R_0805_2012Metric
- SW1: renamed from SW?; footprint (none) -> Button_Switch_THT:SW_PUSH_6mm_H5mm
- Y1: renamed from Y?; footprint (none) -> Crystal:Crystal_SMD_HC49-SD_HandSoldering
- Y2: renamed from Y?; footprint (none) -> Crystal:Crystal_C38-LF_D3.0mm_L8.0mm_Vertical
- gave numbers to parts that had none: 1
Connections:
- net labels added: +3.3VA, CELL_1, CELL_2, CELL_3, ESP_IO0, ESP_RST
- net labels removed: VDDA, VSSA
- wire segments 132 -> 188
Other:
- moved on the sheet: C10, C15, C17, C18, C7, D1, D2, J2, JP1, R1, R2, R3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

Commit message: Layout çizimi tamanlandı.
Layout çizimi ilk şablonu tamamlandı.
Parts:
- removed D4: SD CARD LED, LED_SMD:LED_0805_2012Metric, symbol Device:LED
- removed R6: 470, Resistor_SMD:R_0805_2012Metric, symbol Device:R_Small
- Y1: footprint Crystal:Crystal_SMD_HC49-SD_HandSoldering -> Crystal:Crystal_SMD_HC49-SD
- renumbered C23 to C19, C19 to C20, C20 to C21, R10 to R6, R9 to R7, R7 to R9
Other:
- moved on the sheet: C19, C20

Commit message: Micro Sd kılıf eklendi.
Sd kart holder kılıfı micro sd kart soket kılıfı ile değiştirildi.
Parts:
- removed C3, C4: 10pF, Capacitor_SMD:C_0805_2012Metric, symbol Device:C
- removed J3: Micro_SD_Card_Det_Hirose_DM3AT, Connector_Card:SD_Kyocera_145638009511859+, symbol Connector:Micro_SD_Card_Det_Hirose_DM3AT
- removed Y2: 32K, Crystal:Crystal_C38-LF_D3.0mm_L8.0mm_Vertical, symbol Device:Crystal
- added J3: 693071010811, micro_sd_8+1:micro_sd_8+1, symbol SD_Card_8+1:693071010811
- J1: footprint Connector_JST:JST_XH_B3B-XH-A_1x03_P2.50mm_Vertical -> Connector_PinHeader_2.54mm:PinHeader_1x03_P2.54mm_Vertical
- renumbered C12 to C10, C13 to C11, C14 to C12, C15 to C13, C16 to C14, C17 to C15, C18 to C16, C19 to C17, C20 to C18, C21 to C19, C5 to C3, C6 to C4, C7 to C5, C8 to C6, C9 to C7, C10 to C8, C11 to C9
Connections:
- net labels removed: OSC32_IN, OSC32_OUT
- wire segments 188 -> 173

Commit message: Layout_v2 çizimi tamamlandı.
Parts:
- J3: symbol SD_Card_8+1:693071010811 -> BMS-rescue:693071010811-SD_Card_8+1
Changed lines of the file:
@@
 $EndComp
 $Comp
-L SD_Card_8+1:693071010811 J3
+L BMS-rescue:693071010811-SD_Card_8+1 J3
 U 1 1 60929CF2
 P 9550 4150

Commit message: Çizim tamamlandı.
DRC yapıldı ve hatalar düzeltildi.
Parts:
- added H1, H2, H3, H4: Mounting_Hole, MountingHole:MountingHole_2.2mm_M2_DIN965_Pad, symbol Mechanical:MountingHole
Changed lines of the file:
@@
 Wire Wire Line
 	8900 4250 8900 4800
+$Comp
+L Mechanical:MountingHole H1
+U 1 1 6095B635
+P 7400 5950
+F 0 "H1" H 7500 5996 50  0000 L CNN
+F 1 "Mounting_Hole" H 7500 5905 50  0000 L CNN
+F 2 "MountingHole:MountingHole_2.2mm_M2_DIN965_Pad" H 7400 5950 50  0001 C CNN
+F 3 "~" H 7400 5950 50  0001 C CNN
+	1    7400 5950
+	1    0    0    -1
+$EndComp
+$Comp
+L Mechanical:MountingHole H2
+U 1 1 6095C305
+P 8200 5950
+F 0 "H2" H 8300 5996 50  0000 L CNN
+F 1 "Mounting_Hole" H 8300 5905 50  0000 L CNN
+F 2 "MountingHole:MountingHole_2.2mm_M2_DIN965_Pad" H 8200 5950 50  0001 C CNN
+F 3 "~" H 8200 5950 50  0001 C CNN
+	1    8200 5950
+	1    0    0    -1
+$EndComp
+$Comp
+L Mechanical:MountingHole H3
+U 1 1 609B128C
+P 7400 6150
+F 0 "H3" H 7500 6196 50  0000 L CNN
+F 1 "Mounting_Hole" H 7500 6105 50  0000 L CNN
+F 2 "MountingHole:MountingHole_2.2mm_M2_DIN965_Pad" H 7400 6150 50  0001 C CNN
+F 3 "~" H 7400 6150 50  0001 C CNN
+	1    7400 6150
+	1    0    0    -1
+$EndComp
+$Comp
+L Mechanical:MountingHole H4
+U 1 1 609B9479
+P 8200 6150
+F 0 "H4" H 8300 6196 50  0000 L CNN
+F 1 "Mounting_Hole" H 8300 6105 50  0000 L CNN
+F 2 "MountingHole:MountingHole_2.2mm_M2_DIN965_Pad" H 8200 6150 50  0001 C CNN
+F 3 "~" H 8200 6150 50  0001 C CNN
+	1    8200 6150
+	1    0    0    -1
+$EndComp
 $EndSCHEMATC
